File: Misaka/StepperMotorDriver.sch (KiCad schematic (older format))
At the start: 15 parts, among them J2 Conn_01x04_Male, U1 DRV8825PWPR

Commit message: route v1.1
Connections:
- net at U1.10 (BOUT1): now also J2.1 (Pin_1); no longer J2.2 (Pin_2)
- net at U1.8 (BOUT2): now also J2.2 (Pin_2); no longer J2.1 (Pin_1)
Other:
- moved on the sheet: J2
Changed lines of the file:
@@
 L Connector:Conn_01x04_Male J2
 U 1 1 5E60B6B4
-P 6650 3100
+P 6750 3100
 AR Path="/5E5FA4ED/5E60B6B4" Ref="J2"  Part="1"
 AR Path="/5E601D92/5E60B6B4" Ref="J3"  Part="1"
 AR Path="/5E6050A3/5E60B6B4" Ref="J4"  Part="1"
-F 0 "J2" H 6622 2982 50  0000 R CNN
-F 1 "Conn_01x04_Male" H 6622 3073 50  0000 R CNN
-F 2 "Connector_Molex:Molex_PicoBlade_53047-0410_1x04_P1.25mm_Vertical" H 6650 3100 50  0001 C CNN
-F 3 "~" H 6650 3100 50  0001 C CNN
-	1    6650 3100
+F 0 "J2" H 6722 2982 50  0000 R CNN
+F 1 "Conn_01x04_Male" H 6722 3073 50  0000 R CNN
+F 2 "Connector_Molex:Molex_PicoBlade_53047-0410_1x04_P1.25mm_Vertical" H 6750 3100 50  0001 C CNN
+F 3 "~" H 6750 3100 50  0001 C CNN
+	1    6750 3100
 	-1   0    0    1
 $EndComp
@@
 	5850 4200 5950 4200
 Wire Wire Line
-	6350 2900 6450 2900
-Wire Wire Line
-	6350 3000 6450 3000
-Wire Wire Line
-	6350 3100 6450 3100
-Wire Wire Line
-	6350 3200 6450 3200
+	6350 2900 6550 2900
+Wire Wire Line
+	6350 3000 6550 3000
 Wire Wire Line
 	6350 2800 6700 2800
@@
 Text Label 4450 2750 0    50   ~ 0
 MS1
+Wire Wire Line
+	6350 3100 6450 3100
+Wire Wire Line
+	6450 3100 6450 3200
+Wire Wire Line
+	6450 3200 6550 3200
+Wire Wire Line
+	6350 3200 6400 3200
+Wire Wire Line
+	6400 3200 6400 3150
+Wire Wire Line
+	6400 3150 6500 3150
+Wire Wire Line
+	6500 3150 6500 3100
+Wire Wire Line
+	6500 3100 6550 3100
 $EndSCHEMATC

Commit message: route v2.1
Parts:
- C-VMA1, C-VMB1, C1, C2, C3: footprint Capacitor_SMD:C_0603_1608Metric -> Capacitor_SMD:C_0603_1608Metric_Pad1.05x0.95mm_HandSolder
- CP1: footprint Capacitor_Tantalum_SMD:CP_EIA-1608-08_AVX-J -> Capacitor_Tantalum_SMD:CP_EIA-1608-08_AVX-J_Pad1.25x1.05mm_HandSolder
Changed lines of the file:
@@
 F 0 "C3" H 6615 2296 50  0000 L CNN
 F 1 "0.47uF" H 6615 2205 50  0000 L CNN
-F 2 "Capacitor_SMD:C_0603_1608Metric" H 6538 2100 50  0001 C CNN
+F 2 "Capacitor_SMD:C_0603_1608Metric_Pad1.05x0.95mm_HandSolder" H 6538 2100 50  0001 C CNN
 F 3 "~" H 6500 2250 50  0001 C CNN
 	1    6500 2250
@@
 F 0 "C2" H 5315 2096 50  0000 L CNN
 F 1 "0.1uF" H 5315 2005 50  0000 L CNN
-F 2 "Capacitor_SMD:C_0603_1608Metric" H 5238 1900 50  0001 C CNN
+F 2 "Capacitor_SMD:C_0603_1608Metric_Pad1.05x0.95mm_HandSolder" H 5238 1900 50  0001 C CNN
 F 3 "~" H 5200 2050 50  0001 C CNN
 	1    5200 2050
@@
 F 0 "C1" H 5265 4146 50  0000 L CNN
 F 1 "0.01uF" H 5265 4055 50  0000 L CNN
-F 2 "Capacitor_SMD:C_0603_1608Metric" H 5188 3950 50  0001 C CNN
+F 2 "Capacitor_SMD:C_0603_1608Metric_Pad1.05x0.95mm_HandSolder" H 5188 3950 50  0001 C CNN
 F 3 "~" H 5150 4100 50  0001 C CNN
 	1    5150 4100
@@
 F 0 "C-VMA1" V 6498 3700 50  0000 C CNN
 F 1 "0.1uF" V 6589 3700 50  0000 C CNN
-F 2 "Capacitor_SMD:C_0603_1608Metric" H 6788 3550 50  0001 C CNN
+F 2 "Capacitor_SMD:C_0603_1608Metric_Pad1.05x0.95mm_HandSolder" H 6788 3550 50  0001 C CNN
 F 3 "~" H 6750 3700 50  0001 C CNN
 	1    6750 3700
@@
 F 0 "C-VMB1" V 6498 4150 50  0000 C CNN
 F 1 "0.1uF" V 6589 4150 50  0000 C CNN
-F 2 "Capacitor_SMD:C_0603_1608Metric" H 6788 4000 50  0001 C CNN
+F 2 "Capacitor_SMD:C_0603_1608Metric_Pad1.05x0.95mm_HandSolder" H 6788 4000 50  0001 C CNN
 F 3 "~" H 6750 4150 50  0001 C CNN
 	1    6750 4150
@@
 F 0 "CP1" V 5645 1500 50  0000 C CNN
 F 1 "100uF" V 5736 1500 50  0000 C CNN
-F 2 "Capacitor_Tantalum_SMD:CP_EIA-1608-08_AVX-J" H 5938 1350 50  0001 C CNN
+F 2 "Capacitor_Tantalum_SMD:CP_EIA-1608-08_AVX-J_Pad1.25x1.05mm_HandSolder" H 5938 1350 50  0001 C CNN
 F 3 "~" H 5900 1500 50  0001 C CNN
 	1    5900 1500

Commit message: Change Footprint
Parts:
- CP1: footprint Capacitor_Tantalum_SMD:CP_EIA-1608-08_AVX-J_Pad1.25x1.05mm_HandSolder -> Capacitor_Tantalum_SMD:CP_EIA-3528-21_Kemet-B_Pad1.50x2.35mm_HandSolder
Changed lines of the file:
@@
 F 0 "CP1" V 5645 1500 50  0000 C CNN
 F 1 "100uF" V 5736 1500 50  0000 C CNN
-F 2 "Capacitor_Tantalum_SMD:CP_EIA-1608-08_AVX-J_Pad1.25x1.05mm_HandSolder" H 5938 1350 50  0001 C CNN
+F 2 "Capacitor_Tantalum_SMD:CP_EIA-3528-21_Kemet-B_Pad1.50x2.35mm_HandSolder" H 5938 1350 50  0001 C CNN
 F 3 "~" H 5900 1500 50  0001 C CNN
 	1    5900 1500
