File: Misaka/Power.sch (KiCad schematic (older format))
At the start: 8 parts

Commit message: V1
Parts:
- gave numbers to parts that had none: 8
Changed lines of the file:
@@
 $Descr A4 11693 8268
 encoding utf-8
-Sheet 5 7
+Sheet 5 10
 Title ""
 Date ""
@@
 $EndDescr
 $Comp
-L Device:D D?
+L Device:D D2
 U 1 1 5E62C39C
 P 2300 2000
-F 0 "D?" H 2300 1784 50  0000 C CNN
+F 0 "D2" H 2300 1784 50  0000 C CNN
 F 1 "M7" H 2300 1875 50  0000 C CNN
 F 2 "Diode_SMD:D_SMA_Handsoldering" H 2300 2000 50  0001 C CNN
@@
 $EndComp
 $Comp
-L Device:CP1 CP?
+L Device:CP1 CP4
 U 1 1 5E62F0CC
 P 2600 2350
-F 0 "CP?" H 2715 2396 50  0000 L CNN
+F 0 "CP4" H 2715 2396 50  0000 L CNN
 F 1 "47uF" H 2715 2305 50  0000 L CNN
 F 2 "Capacitor_SMD:CP_Elec_6.3x5.8" H 2600 2350 50  0001 C CNN
@@
 $EndComp
 $Comp
-L Device:C C?
+L Device:C C14
 U 1 1 5E6304AE
 P 3000 2350
-F 0 "C?" H 3115 2396 50  0000 L CNN
+F 0 "C14" H 3115 2396 50  0000 L CNN
 F 1 "100nF" H 3115 2305 50  0000 L CNN
 F 2 "Capacitor_SMD:C_0603_1608Metric_Pad1.05x0.95mm_HandSolder" H 3038 2200 50  0001 C CNN
@@
 $EndComp
 $Comp
-L power:GND #PWR?
+L power:GND #PWR0161
 U 1 1 5E631504
 P 3500 2650
-F 0 "#PWR?" H 3500 2400 50  0001 C CNN
+F 0 "#PWR0161" H 3500 2400 50  0001 C CNN
 F 1 "GND" H 3505 2477 50  0000 C CNN
 F 2 "" H 3500 2650 50  0001 C CNN
@@
 $EndComp
 $Comp
-L Device:CP1 CP?
+L Device:CP1 CP5
 U 1 1 5E638171
 P 4150 2350
-F 0 "CP?" H 4265 2396 50  0000 L CNN
+F 0 "CP5" H 4265 2396 50  0000 L CNN
 F 1 "47uF" H 4265 2305 50  0000 L CNN
 F 2 "Capacitor_SMD:CP_Elec_6.3x5.8" H 4150 2350 50  0001 C CNN
@@
 $EndComp
 $Comp
-L power:+BATT #PWR?
+L power:+BATT #PWR0162
 U 1 1 5E63945A
 P 2000 2000
-F 0 "#PWR?" H 2000 1850 50  0001 C CNN
+F 0 "#PWR0162" H 2000 1850 50  0001 C CNN
 F 1 "+BATT" H 2015 2173 50  0000 C CNN
 F 2 "" H 2000 2000 50  0001 C CNN
@@
 $EndComp
 $Comp
-L power:+5V #PWR?
+L power:+5V #PWR0163
 U 1 1 5E63B921
 P 4300 2000
-F 0 "#PWR?" H 4300 1850 50  0001 C CNN
+F 0 "#PWR0163" H 4300 1850 50  0001 C CNN
 F 1 "+5V" H 4315 2173 50  0000 C CNN
 F 2 "" H 4300 2000 50  0001 C CNN
@@
 Connection ~ 3000 2600
 $Comp
-L Regulator_Linear:AMS1117-3.3 U?
+L Regulator_Linear:AMS1117-3.3 U7
 U 1 1 5E644475
 P 4900 2100
-F 0 "U?" H 4900 2342 50  0000 C CNN
+F 0 "U7" H 4900 2342 50  0000 C CNN
 F 1 "AMS1117-3.3" H 4900 2251 50  0000 C CNN
 F 2 "Package_TO_SOT_SMD:SOT-223-3_TabPin2" H 4900 2300 50  0001 C CNN
@@
 $EndComp
 $Comp
-L Regulator_Linear:AMS1117-5.0 U?
+L Regulator_Linear:AMS1117-5.0 U6
 U 1 1 5E646B9F
 P 3500 2000
-F 0 "U?" H 3500 2242 50  0000 C CNN
+F 0 "U6" H 3500 2242 50  0000 C CNN
 F 1 "AMS1117-5.0" H 3500 2151 50  0000 C CNN
 F 2 "Package_TO_SOT_SMD:SOT-223-3_TabPin2" H 3500 2200 50  0001 C CNN
@@
 	3800 2000 4150 2000
 $Comp
-L power:+5V #PWR?
+L power:+5V #PWR0164
 U 1 1 5E6497A2
 P 4500 2000
-F 0 "#PWR?" H 4500 1850 50  0001 C CNN
+F 0 "#PWR0164" H 4500 1850 50  0001 C CNN
 F 1 "+5V" H 4515 2173 50  0000 C CNN
 F 2 "" H 4500 2000 50  0001 C CNN
@@
 $EndComp
 $Comp
-L power:+3.3V #PWR?
+L power:+3.3V #PWR0165
 U 1 1 5E64AE3C
 P 5300 2000
-F 0 "#PWR?" H 5300 1850 50  0001 C CNN
+F 0 "#PWR0165" H 5300 1850 50  0001 C CNN
 F 1 "+3.3V" H 5315 2173 50  0000 C CNN
 F 2 "" H 5300 2000 50  0001 C CNN
@@
 $EndComp
 $Comp
-L power:GND #PWR?
+L power:GND #PWR0166
 U 1 1 5E64B3E8
 P 4900 2450
-F 0 "#PWR?" H 4900 2200 50  0001 C CNN
+F 0 "#PWR0166" H 4900 2200 50  0001 C CNN
 F 1 "GND" H 4905 2277 50  0000 C CNN
 F 2 "" H 4900 2450 50  0001 C CNN
@@
 	4900 2400 4900 2450
 $Comp
-L Device:LED LED?
+L Device:LED LED1
 U 1 1 5E64FDD4
 P 2750 3050
-F 0 "LED?" H 2743 2795 50  0000 C CNN
+F 0 "LED1" H 2743 2795 50  0000 C CNN
 F 1 "ON" H 2743 2886 50  0000 C CNN
 F 2 "LED_SMD:LED_0603_1608Metric_Pad1.05x0.95mm_HandSolder" H 2750 3050 50  0001 C CNN
@@
 $EndComp
 $Comp
-L Device:R R?
+L Device:R R27
 U 1 1 5E654EE5
 P 2250 3050
-F 0 "R?" V 2043 3050 50  0000 C CNN
+F 0 "R27" V 2043 3050 50  0000 C CNN
 F 1 "1k" V 2134 3050 50  0000 C CNN
 F 2 "Resistor_SMD:R_0603_1608Metric_Pad1.05x0.95mm_HandSolder" V 2180 3050 50  0001 C CNN
@@
 $EndComp
 $Comp
-L power:+5V #PWR?
+L power:+5V #PWR0167
 U 1 1 5E655D03
 P 2000 2950
-F 0 "#PWR?" H 2000 2800 50  0001 C CNN
+F 0 "#PWR0167" H 2000 2800 50  0001 C CNN
 F 1 "+5V" H 2015 3123 50  0000 C CNN
 F 2 "" H 2000 2950 50  0001 C CNN
@@
 $EndComp
 $Comp
-L power:GND #PWR?
+L power:GND #PWR0168
 U 1 1 5E6573BC
 P 3000 3150
-F 0 "#PWR?" H 3000 2900 50  0001 C CNN
+F 0 "#PWR0168" H 3000 2900 50  0001 C CNN
 F 1 "GND" H 3005 2977 50  0000 C CNN
 F 2 "" H 3000 3150 50  0001 C CNN

Commit message: route v2.2
Parts:
- removed LED1: ON, LED_SMD:LED_0603_1608Metric_Pad1.05x0.95mm_HandSolder, symbol Device:LED
- removed R27: 1k, Resistor_SMD:R_0603_1608Metric_Pad1.05x0.95mm_HandSolder, symbol Device:R
Changed lines of the file:
@@
 Wire Wire Line
 	4900 2400 4900 2450
-$Comp
-L Device:LED LED1
-U 1 1 5E64FDD4
-P 2750 3050
-F 0 "LED1" H 2743 2795 50  0000 C CNN
-F 1 "ON" H 2743 2886 50  0000 C CNN
-F 2 "LED_SMD:LED_0603_1608Metric_Pad1.05x0.95mm_HandSolder" H 2750 3050 50  0001 C CNN
-F 3 "~" H 2750 3050 50  0001 C CNN
-	1    2750 3050
-	-1   0    0    1
-$EndComp
-$Comp
-L Device:R R27
-U 1 1 5E654EE5
-P 2250 3050
-F 0 "R27" V 2043 3050 50  0000 C CNN
-F 1 "1k" V 2134 3050 50  0000 C CNN
-F 2 "Resistor_SMD:R_0603_1608Metric_Pad1.05x0.95mm_HandSolder" V 2180 3050 50  0001 C CNN
-F 3 "~" H 2250 3050 50  0001 C CNN
-	1    2250 3050
-	0    1    1    0
-$EndComp
-$Comp
-L power:+5V #PWR0167
-U 1 1 5E655D03
-P 2000 2950
-F 0 "#PWR0167" H 2000 2800 50  0001 C CNN
-F 1 "+5V" H 2015 3123 50  0000 C CNN
-F 2 "" H 2000 2950 50  0001 C CNN
-F 3 "" H 2000 2950 50  0001 C CNN
-	1    2000 2950
-	1    0    0    -1
-$EndComp
-$Comp
-L power:GND #PWR0168
-U 1 1 5E6573BC
-P 3000 3150
-F 0 "#PWR0168" H 3000 2900 50  0001 C CNN
-F 1 "GND" H 3005 2977 50  0000 C CNN
-F 2 "" H 3000 3150 50  0001 C CNN
-F 3 "" H 3000 3150 50  0001 C CNN
-	1    3000 3150
-	1    0    0    -1
-$EndComp
-Wire Wire Line
-	2000 2950 2000 3050
-Wire Wire Line
-	2000 3050 2100 3050
-Wire Wire Line
-	2400 3050 2600 3050
-Wire Wire Line
-	2900 3050 3000 3050
-Wire Wire Line
-	3000 3050 3000 3150
 $EndSCHEMATC
