File: Misaka/Misaka.kicad_pcb (KiCad board)
At the start: 2 copper layers, 100 x 86.6 mm, 104 parts, among them J1 Conn_Coaxial_Power, J2 Conn_01x04_Male, J3 Conn_01x04_Male, J4 Conn_01x04_Male, J5 USB_B_Micro, J6 Conn_01x04_Female, J7 Conn_01x04_Female_UART, J8 Conn_02x04_Odd_Even, J9 Conn_01x07, SW1 SW_DIP_x03, U1 DRV8825PWPR, U2 ATmega2560-16AU, U3 DRV8825PWPR, U4 DRV8825PWPR, U5 CH340C, U6 AMS1117-5.0, U7 AMS1117-3.3, U8 24LC02, Y1 CSTLS16M0X51-B0

Commit message: 电池正负极反了
Parts:
- J1: value Conn_Coaxial_Power -> Battery
Changed lines of the file:
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@@
     (add_net /D10)
     (add_net /D11)
+    (add_net /D12)
     (add_net /D13)
     (add_net /D3)
+    (add_net /D53)
     (add_net /D6)
     (add_net /D7)
@@
     (add_net /RX1)
     (add_net /RX2)
+    (add_net /RX3)
     (add_net /SCK)
     (add_net /SCL)
@@
     (add_net /TX1)
     (add_net /TX2)
+    (add_net /TX3)
     (add_net "Net-(C1-Pad1)")
     (add_net "Net-(C1-Pad2)")
@@
     (add_net "Net-(C7-Pad2)")
     (add_net "Net-(C8-Pad2)")
+    (add_net "Net-(D10-Pad2)")
     (add_net "Net-(D10-Pad4)")
     (add_net "Net-(D3-Pad2)")
@@
     (add_net "Net-(J5-Pad2)")
     (add_net "Net-(J5-Pad3)")
+    (add_net "Net-(J5-Pad4)")
     (add_net "Net-(J7-Pad3)")
     (add_net "Net-(J7-Pad4)")
+    (add_net "Net-(J8-Pad6)")
     (add_net "Net-(L1-Pad2)")
+    (add_net "Net-(MOD1-Pad11)")
+    (add_net "Net-(MOD1-Pad12)")
+    (add_net "Net-(MOD1-Pad13)")
+    (add_net "Net-(MOD1-Pad14)")
+    (add_net "Net-(MOD1-Pad15)")
+    (add_net "Net-(MOD1-Pad16)")
+    (add_net "Net-(MOD1-Pad17)")
+    (add_net "Net-(MOD1-Pad18)")
+    (add_net "Net-(MOD1-Pad19)")
+    (add_net "Net-(MOD1-Pad20)")
+    (add_net "Net-(MOD1-Pad4)")
+    (add_net "Net-(MOD1-Pad5)")
+    (add_net "Net-(MOD1-Pad6)")
+    (add_net "Net-(MOD1-Pad7)")
+    (add_net "Net-(MOD1-Pad8)")
+    (add_net "Net-(MOD1-Pad9)")
     (add_net "Net-(R11-Pad1)")
     (add_net "Net-(R12-Pad1)")
@@
     (add_net "Net-(R7-Pad1)")
     (add_net "Net-(R8-Pad2)")
+    (add_net "Net-(U1-Pad19)")
+    (add_net "Net-(U1-Pad21)")
+    (add_net "Net-(U1-Pad23)")
+    (add_net "Net-(U2-Pad1)")
+    (add_net "Net-(U2-Pad14)")
+    (add_net "Net-(U2-Pad27)")
+    (add_net "Net-(U2-Pad28)")
+    (add_net "Net-(U2-Pad29)")
+    (add_net "Net-(U2-Pad35)")
+    (add_net "Net-(U2-Pad36)")
+    (add_net "Net-(U2-Pad37)")
+    (add_net "Net-(U2-Pad38)")
+    (add_net "Net-(U2-Pad39)")
+    (add_net "Net-(U2-Pad4)")
+    (add_net "Net-(U2-Pad40)")
+    (add_net "Net-(U2-Pad41)")
+    (add_net "Net-(U2-Pad42)")
+    (add_net "Net-(U2-Pad47)")
+    (add_net "Net-(U2-Pad48)")
+    (add_net "Net-(U2-Pad49)")
+    (add_net "Net-(U2-Pad5)")
+    (add_net "Net-(U2-Pad50)")
+    (add_net "Net-(U2-Pad51)")
+    (add_net "Net-(U2-Pad52)")
+    (add_net "Net-(U2-Pad53)")
+    (add_net "Net-(U2-Pad54)")
+    (add_net "Net-(U2-Pad55)")
+    (add_net "Net-(U2-Pad56)")
+    (add_net "Net-(U2-Pad57)")
+    (add_net "Net-(U2-Pad58)")
+    (add_net "Net-(U2-Pad59)")
+    (add_net "Net-(U2-Pad6)")
+    (add_net "Net-(U2-Pad60)")
+    (add_net "Net-(U2-Pad65)")
+    (add_net "Net-(U2-Pad66)")
+    (add_net "Net-(U2-Pad67)")
+    (add_net "Net-(U2-Pad68)")
+    (add_net "Net-(U2-Pad69)")
+    (add_net "Net-(U2-Pad70)")
+    (add_net "Net-(U2-Pad71)")
+    (add_net "Net-(U2-Pad72)")
+    (add_net "Net-(U2-Pad73)")
+    (add_net "Net-(U2-Pad74)")
+    (add_net "Net-(U2-Pad75)")
+    (add_net "Net-(U2-Pad76)")
+    (add_net "Net-(U2-Pad77)")
+    (add_net "Net-(U2-Pad78)")
+    (add_net "Net-(U2-Pad79)")
+    (add_net "Net-(U2-Pad8)")
+    (add_net "Net-(U2-Pad82)")
+    (add_net "Net-(U2-Pad83)")
+    (add_net "Net-(U2-Pad84)")
+    (add_net "Net-(U2-Pad85)")
+    (add_net "Net-(U2-Pad86)")
+    (add_net "Net-(U2-Pad87)")
+    (add_net "Net-(U2-Pad88)")
+    (add_net "Net-(U2-Pad89)")
+    (add_net "Net-(U2-Pad9)")
+    (add_net "Net-(U2-Pad90)")
+    (add_net "Net-(U2-Pad91)")
+    (add_net "Net-(U2-Pad92)")
+    (add_net "Net-(U2-Pad93)")
+    (add_net "Net-(U2-Pad94)")
+    (add_net "Net-(U2-Pad95)")
+    (add_net "Net-(U2-Pad96)")
+    (add_net "Net-(U2-Pad97)")
+    (add_net "Net-(U2-Pad98)")
+    (add_net "Net-(U3-Pad19)")
+    (add_net "Net-(U3-Pad21)")
+    (add_net "Net-(U3-Pad23)")
+    (add_net "Net-(U4-Pad19)")
+    (add_net "Net-(U4-Pad21)")
+    (add_net "Net-(U4-Pad23)")
+    (add_net "Net-(U5-Pad10)")
+    (add_net "Net-(U5-Pad11)")
+    (add_net "Net-(U5-Pad12)")
+    (add_net "Net-(U5-Pad14)")
+    (add_net "Net-(U5-Pad15)")
+    (add_net "Net-(U5-Pad7)")
+    (add_net "Net-(U5-Pad8)")
+    (add_net "Net-(U5-Pad9)")
   )
   (net_class Power ""
@@
       (effects (font (size 1 1) (thickness 0.15)))
     )
-    (fp_text value Conn_Coaxial_Power (at -2.5 3.5) (layer F.Fab)
+    (fp_text value Battery (at -2.5 3.5) (layer F.Fab)
       (effects (font (size 1 1) (thickness 0.15)))
     )

Commit message: 5V-problem
Routing:
- net +5V: track 463.2 -> 578.2 mm, vias 12 -> 13
Changed lines of the file:
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@@
     (thickness 1.6)
     (drawings 9)
-    (tracks 1519)
+    (tracks 1536)
     (zones 0)
     (modules 104)
@@
   )
   (setup
-    (last_trace_width 0.254)
+    (last_trace_width 0.508)
     (user_trace_width 0.127)
     (user_trace_width 0.254)
@@
     (add_net /D10)
     (add_net /D11)
-    (add_net /D12)
     (add_net /D13)
     (add_net /D3)
-    (add_net /D53)
     (add_net /D6)
     (add_net /D7)
@@
     (add_net /RX1)
     (add_net /RX2)
-    (add_net /RX3)
     (add_net /SCK)
     (add_net /SCL)
@@
     (add_net /TX1)
     (add_net /TX2)
-    (add_net /TX3)
     (add_net "Net-(C1-Pad1)")
     (add_net "Net-(C1-Pad2)")
@@
     (add_net "Net-(C7-Pad2)")
     (add_net "Net-(C8-Pad2)")
-    (add_net "Net-(D10-Pad2)")
     (add_net "Net-(D10-Pad4)")
     (add_net "Net-(D3-Pad2)")
@@
     (add_net "Net-(J5-Pad2)")
     (add_net "Net-(J5-Pad3)")
-    (add_net "Net-(J5-Pad4)")
     (add_net "Net-(J7-Pad3)")
     (add_net "Net-(J7-Pad4)")
-    (add_net "Net-(J8-Pad6)")
     (add_net "Net-(L1-Pad2)")
-    (add_net "Net-(MOD1-Pad11)")
-    (add_net "Net-(MOD1-Pad12)")
-    (add_net "Net-(MOD1-Pad13)")
-    (add_net "Net-(MOD1-Pad14)")
-    (add_net "Net-(MOD1-Pad15)")
-    (add_net "Net-(MOD1-Pad16)")
-    (add_net "Net-(MOD1-Pad17)")
-    (add_net "Net-(MOD1-Pad18)")
-    (add_net "Net-(MOD1-Pad19)")
-    (add_net "Net-(MOD1-Pad20)")
-    (add_net "Net-(MOD1-Pad4)")
-    (add_net "Net-(MOD1-Pad5)")
-    (add_net "Net-(MOD1-Pad6)")
-    (add_net "Net-(MOD1-Pad7)")
-    (add_net "Net-(MOD1-Pad8)")
-    (add_net "Net-(MOD1-Pad9)")
     (add_net "Net-(R11-Pad1)")
     (add_net "Net-(R12-Pad1)")
@@
     (add_net "Net-(R7-Pad1)")
     (add_net "Net-(R8-Pad2)")
-    (add_net "Net-(U1-Pad19)")
-    (add_net "Net-(U1-Pad21)")
-    (add_net "Net-(U1-Pad23)")
-    (add_net "Net-(U2-Pad1)")
-    (add_net "Net-(U2-Pad14)")
-    (add_net "Net-(U2-Pad27)")
-    (add_net "Net-(U2-Pad28)")
-    (add_net "Net-(U2-Pad29)")
-    (add_net "Net-(U2-Pad35)")
-    (add_net "Net-(U2-Pad36)")
-    (add_net "Net-(U2-Pad37)")
-    (add_net "Net-(U2-Pad38)")
-    (add_net "Net-(U2-Pad39)")
-    (add_net "Net-(U2-Pad4)")
-    (add_net "Net-(U2-Pad40)")
-    (add_net "Net-(U2-Pad41)")
-    (add_net "Net-(U2-Pad42)")
-    (add_net "Net-(U2-Pad47)")
-    (add_net "Net-(U2-Pad48)")
-    (add_net "Net-(U2-Pad49)")
-    (add_net "Net-(U2-Pad5)")
-    (add_net "Net-(U2-Pad50)")
-    (add_net "Net-(U2-Pad51)")
-    (add_net "Net-(U2-Pad52)")
-    (add_net "Net-(U2-Pad53)")
-    (add_net "Net-(U2-Pad54)")
-    (add_net "Net-(U2-Pad55)")
-    (add_net "Net-(U2-Pad56)")
-    (add_net "Net-(U2-Pad57)")
-    (add_net "Net-(U2-Pad58)")
-    (add_net "Net-(U2-Pad59)")
-    (add_net "Net-(U2-Pad6)")
-    (add_net "Net-(U2-Pad60)")
-    (add_net "Net-(U2-Pad65)")
-    (add_net "Net-(U2-Pad66)")
-    (add_net "Net-(U2-Pad67)")
-    (add_net "Net-(U2-Pad68)")
-    (add_net "Net-(U2-Pad69)")
-    (add_net "Net-(U2-Pad70)")
-    (add_net "Net-(U2-Pad71)")
-    (add_net "Net-(U2-Pad72)")
-    (add_net "Net-(U2-Pad73)")
-    (add_net "Net-(U2-Pad74)")
-    (add_net "Net-(U2-Pad75)")
-    (add_net "Net-(U2-Pad76)")
-    (add_net "Net-(U2-Pad77)")
-    (add_net "Net-(U2-Pad78)")
-    (add_net "Net-(U2-Pad79)")
-    (add_net "Net-(U2-Pad8)")
-    (add_net "Net-(U2-Pad82)")
-    (add_net "Net-(U2-Pad83)")
-    (add_net "Net-(U2-Pad84)")
-    (add_net "Net-(U2-Pad85)")
-    (add_net "Net-(U2-Pad86)")
-    (add_net "Net-(U2-Pad87)")
-    (add_net "Net-(U2-Pad88)")
-    (add_net "Net-(U2-Pad89)")
-    (add_net "Net-(U2-Pad9)")
-    (add_net "Net-(U2-Pad90)")
-    (add_net "Net-(U2-Pad91)")
-    (add_net "Net-(U2-Pad92)")
-    (add_net "Net-(U2-Pad93)")
-    (add_net "Net-(U2-Pad94)")
-    (add_net "Net-(U2-Pad95)")
-    (add_net "Net-(U2-Pad96)")
-    (add_net "Net-(U2-Pad97)")
-    (add_net "Net-(U2-Pad98)")
-    (add_net "Net-(U3-Pad19)")
-    (add_net "Net-(U3-Pad21)")
-    (add_net "Net-(U3-Pad23)")
-    (add_net "Net-(U4-Pad19)")
-    (add_net "Net-(U4-Pad21)")
-    (add_net "Net-(U4-Pad23)")
-    (add_net "Net-(U5-Pad10)")
-    (add_net "Net-(U5-Pad11)")
-    (add_net "Net-(U5-Pad12)")
-    (add_net "Net-(U5-Pad14)")
-    (add_net "Net-(U5-Pad15)")
-    (add_net "Net-(U5-Pad7)")
-    (add_net "Net-(U5-Pad8)")
-    (add_net "Net-(U5-Pad9)")
   )
   (net_class Power ""
@@
   (segment (start 59.875 59.925) (end 58.96498 59.01498) (width 0.254) (layer F.Cu) (net 16))
   (segment (start 59.875 60.4) (end 59.875 59.925) (width 0.254) (layer F.Cu) (net 16))
-  (segment (start 60.86751 65.567394) (end 58.994904 67.44) (width 0.127) (layer F.Cu) (net 16))
-  (segment (start 60.86751 61.86751) (end 60.86751 65.567394) (width 0.127) (layer F.Cu) (net 16))
   (segment (start 59.875 60.4) (end 59.875 60.875) (width 0.127) (layer F.Cu) (net 16))
-  (segment (start 59.875 60.875) (end 60.86751 61.86751) (width 0.127) (layer F.Cu) (net 16))
   (segment (start 58 68.2) (end 58 68.9375) (width 0.127) (layer F.Cu) (net 16))
-  (segment (start 58.68 67.44) (end 58 68.12) (width 0.127) (layer F.Cu) (net 16))
   (segment (start 58 68.12) (end 58 68.2) (width 0.127) (layer F.Cu) (net 16))
-  (segment (start 58.994904 67.44) (end 58.68 67.44) (width 0.127) (layer F.Cu) (net 16))
   (via (at 60.88 58.81) (size 0.6) (drill 0.3) (layers F.Cu B.Cu) (net 16))
   (segment (start 59.875 60.4) (end 59.875 59.815) (width 0.254) (layer F.Cu) (net 16))
@@
   (segment (start 94.488 43.415) (end 95.504 42.399) (width 0.254) (layer B.Cu) (net 16))
   (segment (start 95.504 42.399) (end 95.504 41.148) (width 0.254) (layer B.Cu) (net 16))
-  (segment (start 95.504 40.723736) (end 98.127736 38.1) (width 0.254) (layer F.Cu) (net 16))
   (segment (start 95.504 41.148) (end 95.504 40.723736) (width 0.254) (layer F.Cu) (net 16))
-  (segment (start 98.127736 38.1) (end 100.584 38.1) (width 0.254) (layer F.Cu) (net 16))
-  (segment (start 102.34 39.856) (end 102.34 48.45) (width 0.254) (layer F.Cu) (net 16))
-  (segment (start 100.584 38.1) (end 102.34 39.856) (width 0.254) (layer F.Cu) (net 16))
   (segment (start 94.798 82.023) (end 94.798 82.673) (width 0.254) (layer B.Cu) (net 16))
   (via (at 96.52 80.772) (size 0.6) (drill 0.3) (layers F.Cu B.Cu) (net 16))
@@
   (segment (start 100.874 100.076) (end 102.34 98.61) (width 0.508) (layer F.Cu) (net 16))
   (segment (start 100.33 100.076) (end 100.874 100.076) (width 0.508) (layer F.Cu) (net 16))
+  (via (at 55.2 61.9) (size 1.2) (drill 0.7) (layers F.Cu B.Cu) (net 16))
+  (segment (start 53.6125 64.3) (end 53.6125 63.4875) (width 0.5) (layer F.Cu) (net 16))
+  (segment (start 53.6125 63.4875) (end 55.2 61.9) (width 0.5) (layer F.Cu) (net 16))
+  (segment (start 63.765 61.9) (end 64.425 61.24) (width 0.5) (layer B.Cu) (net 16))
+  (segment (start 55.2 61.9) (end 63.765 61.9) (width 0.5) (layer B.Cu) (net 16))
+  (segment (start 70.6 33) (end 71.9 34.3) (width 0.5) (layer F.Cu) (net 16))
+  (segment (start 71.9 34.3) (end 71.9 37.5) (width 0.5) (layer F.Cu) (net 16))
+  (segment (start 66.725 34.325) (end 68.05 33) (width 0.5) (layer F.Cu) (net 16))
+  (segment (start 94.3 37.5) (end 96.5 39.7) (width 0.5) (layer F.Cu) (net 16))
+  (segment (start 95.504 40.723736) (end 96.5 39.7) (width 0.254) (layer F.Cu) (net 16))
+  (segment (start 71.9 37.5) (end 94.3 37.5) (width 0.5) (layer F.Cu) (net 16))
+  (segment (start 66.725 34.8) (end 66.725 34.325) (width 0.5) (layer F.Cu) (net 16))
+  (segment (start 68.05 33) (end 70.6 33) (width 0.5) (layer F.Cu) (net 16))
+  (segment (start 96.5 39.7) (end 96.5 39.6) (width 0.508) (layer F.Cu) (net 16))
+  (segment (start 96.5 39.6) (end 97.5 38.6) (width 0.508) (layer F.Cu) (net 16))
+  (segment (start 97.5 38.6) (end 99.6 38.6) (width 0.508) (layer F.Cu) (net 16))
+  (segment (start 102.34 41.34) (end 102.34 48.45) (width 0.508) (layer F.Cu) (net 16))
+  (segment (start 99.6 38.6) (end 102.34 41.34) (width 0.508) (layer F.Cu) (net 16))
+  (segment (start 79.883999 111.951999) (end 79.992 112.06) (width 0.508) (layer F.Cu) (net 16))
+  (segment (start 53.669863 111.951999) (end 79.883999 111.951999) (width 0.508) (layer F.Cu) (net 16))
+  (segment (start 45.966011 104.248147) (end 53.669863 111.951999) (width 0.508) (layer F.Cu) (net 16))
+  (segment (start 45.966011 86.967972) (end 45.966011 104.248147) (width 0.508) (layer F.Cu) (net 16))
+  (segment (start 42.302412 83.304373) (end 45.966011 86.967972) (width 0.508) (layer F.Cu) (net 16))
+  (segment (start 79.992 112.06) (end 82.4 112.06) (width 0.508) (layer F.Cu) (net 16))
+  (segment (start 35.264373 83.304373) (end 42.302412 83.304373) (width 0.508) (layer F.Cu) (net 16))
+  (segment (start 29.56 77.6) (end 35.264373 83.304373) (width 0.508) (layer F.Cu) (net 16))
   (segment (start 60.89 49.45) (end 60.775 49.565) (width 0.508) (layer F.Cu) (net 17))
   (segment (start 65.7 49.45) (end 60.89 49.45) (width 0.508) (layer F.Cu) (net 17))
@@
     (connect_pads (clearance 0.508))
     (min_thickness 0.254)
-    (fill yes (arc_segments 32) (thermal_gap 0.508) (thermal_bridge_width 0.508))
+    (fill (arc_segments 32) (thermal_gap 0.508) (thermal_bridge_width 0.508))
     (polygon
       (pts
@@
     (connect_pads (clearance 0.508))
     (min_thickness 0.254)
-    (fill yes (arc_segments 32) (thermal_gap 0.508) (thermal_bridge_width 0.508))
+    (fill (arc_segments 32) (thermal_gap 0.508) (thermal_bridge_width 0.508))
     (polygon
       (pts
